File: optiplower.kicad_sch (KiCad schematic)
At the start: 22 parts, among them J1 Conn_01x02, J2 Conn_01x03, U1 LR7533-M, U2 XL4015, U3 DS2502, U4 ATtiny25-20SSN, U5 ATtiny85-20PU, U6 DS2502S+

Commit message: Correct ATTiny PN
Parts:
- U4: value ATtiny25-20SSN -> ATtiny25-20SSU; Farnell PN 2774976 -> 1636951; LCSC C1339960 -> C1338203; MPN ATtiny25-20SSN -> ATtiny25-20SSU
Changed lines of the file:
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@@
       (effects (font (size 1.27 1.27)) (justify right))
     )
-    (property "Value" "ATtiny25-20SSN" (at 128.27 99.695 0)
+    (property "Value" "ATtiny25-20SSU" (at 128.27 99.695 0)
       (effects (font (size 1.27 1.27)) (justify right))
     )
@@
       (effects (font (size 1.27 1.27)) hide)
     )
-    (property "LCSC" "C1339960" (at 142.24 97.79 0)
+    (property "LCSC" "C1338203" (at 142.24 97.79 0)
       (effects (font (size 1.27 1.27)) hide)
     )
-    (property "MPN" "ATtiny25-20SSN" (at 142.24 97.79 0)
+    (property "MPN" "ATtiny25-20SSU" (at 142.24 97.79 0)
       (effects (font (size 1.27 1.27)) hide)
     )
@@
       (effects (font (size 1.27 1.27)) hide)
     )
-    (property "Farnell PN" "2774976" (at 142.24 97.79 0)
+    (property "Farnell PN" "1636951" (at 142.24 97.79 0)
       (effects (font (size 1.27 1.27)) hide)
     )
