File: optiplower.kicad_sch (KiCad schematic)
At the start: 22 parts, among them J1 Conn_01x02, J2 Conn_01x03, U1 LR7533-M, U2 XL4015, U3 DS2502, U4 ATtiny25-20SSU, U5 ATtiny85-20PU, U6 DS2502S+

Commit message: Messing around trying to get timings right in PulseView
Parts:
- U1: now not fitted; now left out of the parts list
- U4: value ATtiny25-20SSU -> ATtiny25-10SSU; Farnell PN 1636951 -> 1636952; LCSC C1338203 -> C148097; MPN ATtiny25-20SSU -> ATtiny25-10SSU
Connections:
- net +3V3: no longer U1.2 (VO)
- net GND: no longer U1.1 (GND)
- net VCC: no longer U1.3 (VI)
Other:
- note added: "Testing shows ATTiny should be run at 2.7v This is a 3v3 part"
- moved on the sheet: U3
Changed lines of the file:
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@@
   (junction (at 77.47 31.75) (diameter 0) (color 0 0 0 0)
   )
-  (junction (at 227.33 46.99) (diameter 0) (color 0 0 0 0)
-  )
   (junction (at 149.86 57.15) (diameter 0) (color 0 0 0 0)
   )
@@
   (junction (at 180.34 50.8) (diameter 0) (color 0 0 0 0)
   )
-  (junction (at 99.06 102.87) (diameter 0) (color 0 0 0 0)
+  (junction (at 85.09 105.41) (diameter 0) (color 0 0 0 0)
   )
   (junction (at 149.86 31.75) (diameter 0) (color 0 0 0 0)
@@
     (stroke (width 0) (type default))
   )
-  (wire (pts (xy 99.06 102.87) (xy 99.06 109.22))
+  (wire (pts (xy 85.09 105.41) (xy 85.09 111.76))
     (stroke (width 0) (type default))
   )
@@
     (stroke (width 0) (type default))
   )
-  (wire (pts (xy 90.17 104.14) (xy 96.52 104.14))
+  (wire (pts (xy 76.2 106.68) (xy 82.55 106.68))
     (stroke (width 0) (type default))
   )
@@
     (stroke (width 0) (type default))
   )
-  (wire (pts (xy 96.52 102.87) (xy 96.52 104.14))
+  (wire (pts (xy 82.55 105.41) (xy 82.55 106.68))
     (stroke (width 0) (type default))
   )
@@
     (stroke (width 0) (type default))
   )
-  (wire (pts (xy 99.06 102.87) (xy 101.6 102.87))
+  (wire (pts (xy 85.09 105.41) (xy 87.63 105.41))
     (stroke (width 0) (type default))
   )
@@
   (wire (pts (xy 139.7 31.75) (xy 149.86 31.75))
     (stroke (width 0) (type default))
+  )
+  (text "Testing shows ATTiny should be run at 2.7v\nThis is a 3v3 part"
+    (at 273.05 29.21 0)
+    (effects (font (size 1.27 1.27)) (justify left bottom))
   )
   (text "Adjustability from 18.29v - 20.125v" (at 120.65 62.23 0)
@@
     (effects (font (size 1.27 1.27)) (justify right bottom))
   )
-  (label "SENSE" (at 90.17 104.14 180) (fields_autoplaced)
+  (label "SENSE" (at 76.2 106.68 180) (fields_autoplaced)
     (effects (font (size 1.27 1.27)) (justify right bottom))
   )
@@
       (effects (font (size 1.27 1.27)) (justify right))
     )
-    (property "Value" "ATtiny25-20SSU" (at 128.27 99.695 0)
+    (property "Value" "ATtiny25-10SSU" (at 128.27 99.695 0)
       (effects (font (size 1.27 1.27)) (justify right))
     )
@@
       (effects (font (size 1.27 1.27)) hide)
     )
-    (property "LCSC" "C1338203" (at 142.24 97.79 0)
-      (effects (font (size 1.27 1.27)) hide)
-    )
-    (property "MPN" "ATtiny25-20SSU" (at 142.24 97.79 0)
+    (property "LCSC" "C148097" (at 142.24 97.79 0)
+      (effects (font (size 1.27 1.27)) hide)
+    )
+    (property "MPN" "ATtiny25-10SSU" (at 142.24 97.79 0)
       (effects (font (size 1.27 1.27)) hide)
     )
@@
       (effects (font (size 1.27 1.27)) hide)
     )
-    (property "Farnell PN" "1636951" (at 142.24 97.79 0)
+    (property "Farnell PN" "1636952" (at 142.24 97.79 0)
       (effects (font (size 1.27 1.27)) hide)
     )
@@
     )
   )
-  (symbol (lib_id "power:GND") (at 99.06 109.22 0) (unit 1)
-    (in_bom yes) (on_board yes) (dnp no) (fields_autoplaced)
-    (property "Reference" "#PWR08" (at 99.06 115.57 0)
-      (effects (font (size 1.27 1.27)) hide)
-    )
-    (property "Value" "GND" (at 99.06 114.3 0)
-      (effects (font (size 1.27 1.27)))
-    )
-    (property "Footprint" "" (at 99.06 109.22 0)
-      (effects (font (size 1.27 1.27)) hide)
-    )
-    (property "Datasheet" "" (at 99.06 109.22 0)
+  (symbol (lib_id "power:GND") (at 85.09 111.76 0) (unit 1)
+    (in_bom yes) (on_board yes) (dnp no) (fields_autoplaced)
+    (property "Reference" "#PWR08" (at 85.09 118.11 0)
+      (effects (font (size 1.27 1.27)) hide)
+    )
+    (property "Value" "GND" (at 85.09 116.84 0)
+      (effects (font (size 1.27 1.27)))
+    )
+    (property "Footprint" "" (at 85.09 111.76 0)
+      (effects (font (size 1.27 1.27)) hide)
+    )
+    (property "Datasheet" "" (at 85.09 111.76 0)
       (effects (font (size 1.27 1.27)) hide)
     )
@@
     )
   )
-  (symbol (lib_id "Optiplower:DS2502") (at 99.06 96.52 0) (unit 1)
+  (symbol (lib_id "Optiplower:DS2502") (at 85.09 99.06 0) (unit 1)
     (in_bom no) (on_board yes) (dnp yes) (fields_autoplaced)
-    (property "Reference" "U3" (at 105.41 96.52 0)
-      (effects (font (size 1.27 1.27)) (justify left))
-    )
-    (property "Value" "DS2502" (at 105.41 99.06 0)
-      (effects (font (size 1.27 1.27)) (justify left))
-    )
-    (property "Footprint" "Package_TO_SOT_THT:TO-92_Inline" (at 99.06 96.52 0)
-      (effects (font (size 1.27 1.27)) hide)
-    )
-    (property "Datasheet" "https://www.analog.com/media/en/technical-documentation/data-sheets/DS2502.pdf" (at 99.06 96.52 0)
-      (effects (font (size 1.27 1.27)) hide)
-    )
-    (property "MPN" "" (at 99.06 96.52 0)
-      (effects (font (size 1.27 1.27)) hide)
-    )
-    (property "Manufacturer" "" (at 99.06 96.52 0)
+    (property "Reference" "U3" (at 91.44 99.06 0)
+      (effects (font (size 1.27 1.27)) (justify left))
+    )
+    (property "Value" "DS2502" (at 91.44 101.6 0)
+      (effects (font (size 1.27 1.27)) (justify left))
+    )
+    (property "Footprint" "Package_TO_SOT_THT:TO-92_Inline" (at 85.09 99.06 0)
+      (effects (font (size 1.27 1.27)) hide)
+    )
+    (property "Datasheet" "https://www.analog.com/media/en/technical-documentation/data-sheets/DS2502.pdf" (at 85.09 99.06 0)
+      (effects (font (size 1.27 1.27)) hide)
+    )
+    (property "MPN" "" (at 85.09 99.06 0)
+      (effects (font (size 1.27 1.27)) hide)
+    )
+    (property "Manufacturer" "" (at 85.09 99.06 0)
       (effects (font (size 1.27 1.27)) hide)
     )
@@
     )
   )
-  (symbol (lib_id "Regulator_Linear:AZ1117-3.3") (at 227.33 39.37 0) (unit 1)
-    (in_bom yes) (on_board yes) (dnp no) (fields_autoplaced)
-    (property "Reference" "U1" (at 227.33 33.02 0)
-      (effects (font (size 1.27 1.27)))
-    )
-    (property "Value" "LR7533-M" (at 227.33 35.56 0)
-      (effects (font (size 1.27 1.27)))
-    )
-    (property "Footprint" "Package_TO_SOT_SMD:SOT-89-3_Handsoldering" (at 227.33 33.02 0)
+  (symbol (lib_id "Regulator_Linear:AZ1117-3.3") (at 264.16 25.4 0) (unit 1)
+    (in_bom no) (on_board no) (dnp yes) (fields_autoplaced)
+    (property "Reference" "U1" (at 264.16 19.05 0)
+      (effects (font (size 1.27 1.27)))
+    )
+    (property "Value" "LR7533-M" (at 264.16 21.59 0)
+      (effects (font (size 1.27 1.27)))
+    )
+    (property "Footprint" "Package_TO_SOT_SMD:SOT-89-3_Handsoldering" (at 264.16 19.05 0)
       (effects (font (size 1.27 1.27) italic) hide)
     )
-    (property "Datasheet" "" (at 227.33 39.37 0)
-      (effects (font (size 1.27 1.27)) hide)
-    )
-    (property "LCSC" "C486076" (at 227.33 39.37 0)
-      (effects (font (size 1.27 1.27)) hide)
-    )
-    (property "MPN" "LR7533-M" (at 227.33 39.37 0)
-      (effects (font (size 1.27 1.27)) hide)
-    )
-    (property "Manufacturer" "LR" (at 227.33 39.37 0)
-      (effects (font (size 1.27 1.27)) hide)
-    )
+    (property "Datasheet" "" (at 264.16 25.4 0)
+      (effects (font (size 1.27 1.27)) hide)
+    )
+    (property "LCSC" "C486076" (at 264.16 25.4 0)
+      (effects (font (size 1.27 1.27)) hide)
+    )
+    (property "MPN" "LR7533-M" (at 264.16 25.4 0)
+      (effects (font (size 1.27 1.27)) hide)
+    )
+    (property "Manufacturer" "LR" (at 264.16 25.4 0)
+      (effects (font (size 1.27 1.27)) hide)
+    )
