File: Programmer/Programmer.kicad_sch (KiCad schematic)
At the start: 10 parts, among them J1 Conn_01x04, J2 Conn_01x03, Q5 LBSS84LT1G, Q7 2N7002

Commit message: LCSC parts
Parts:
- added Q5: LBSS84LT1G, Package_TO_SOT_SMD:SOT-23, symbol Transistor_FET:BSS84
- C2: LCSC (none) -> C1620
- Q5: value LBSS84LT1G -> AO3401A; Farnell PN 1972673 -> 2061518; LCSC C8492 -> C15127
- R5: LCSC (none) -> C23162
- R6, R7: LCSC (none) -> C25197
Changed lines of the file:
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@@
+      (effects (font (size 1.27 1.27)) hide)
+    )
+    (property "LCSC" "C1620" (at 152.4 106.68 0)
       (effects (font (size 1.27 1.27)) hide)
     )
@@
       (effects (font (size 1.27 1.27)) hide)
     )
+    (property "LCSC" "C25197" (at 143.51 78.74 0)
+      (effects (font (size 1.27 1.27)) hide)
+    )
     (pin "1")
     (pin "2")
@@
     )
     (property "Datasheet" "~" (at 125.9428 84.2894 0)
+      (effects (font (size 1.27 1.27)) hide)
+    )
+    (property "LCSC" "C25197" (at 125.9428 84.2894 0)
       (effects (font (size 1.27 1.27)) hide)
     )
@@
       (effects (font (size 1.27 1.27)) hide)
     )
+    (property "LCSC" "C23162" (at 102.87 85.09 0)
+      (effects (font (size 1.27 1.27)) hide)
+    )
     (pin "1")
     (pin "2")
@@
         (path "/cd079a96-fb69-4071-9ed9-61ba2e24ca2f"
           (reference "R1") (unit 1)
+        )
+      )
+    )
+  )
+  (symbol (lib_id "Transistor_FET:BSS84") (at 245.11 50.8 0) (mirror x) (unit 1)
+    (in_bom no) (on_board no) (dnp yes)
+    (property "Reference" "Q5" (at 251.46 51.435 0)
+      (effects (font (size 1.27 1.27)) (justify left))
+    )
+    (property "Value" "LBSS84LT1G" (at 251.46 48.895 0)
+      (effects (font (size 1.27 1.27)) (justify left))
+    )
+    (property "Footprint" "Package_TO_SOT_SMD:SOT-23" (at 250.19 48.895 0)
+      (effects (font (size 1.27 1.27) italic) (justify left) hide)
+    )
+    (property "Datasheet" "http://assets.nexperia.com/documents/data-sheet/BSS84.pdf" (at 245.11 50.8 0)
+      (effects (font (size 1.27 1.27)) (justify left) hide)
+    )
+    (property "LCSC" "C8492" (at 245.11 50.8 0)
+      (effects (font (size 1.27 1.27)) hide)
+    )
+    (property "Farnell PN" "1972673" (at 245.11 50.8 0)
+      (effects (font (size 1.27 1.27)) hide)
+    )
+    (pin "1")
+    (pin "2")
+    (pin "3")
+    (instances
+      (project "DS2502_prog"
+        (path "/0cb1b2db-3266-4f9c-b606-aeea0b5a2127"
+          (reference "Q5") (unit 1)
+        )
+      )
+      (project "Programmer"
+        (path "/cd079a96-fb69-4071-9ed9-61ba2e24ca2f"
+          (reference "Q5") (unit 1)
         )
       )
@@
       (effects (font (size 1.27 1.27)) (justify left))
     )
-    (property "Value" "LBSS84LT1G" (at 157.48 86.995 0)
+    (property "Value" "AO3401A" (at 157.48 86.995 0)
       (effects (font (size 1.27 1.27)) (justify left))
     )
@@
       (effects (font (size 1.27 1.27) italic) (justify left) hide)
     )
-    (property "Datasheet" "http://assets.nexperia.com/documents/data-sheet/BSS84.pdf" (at 151.13 88.9 0)
-      (effects (font (size 1.27 1.27)) (justify left) hide)
-    )
-    (property "LCSC" "C8492" (at 151.13 88.9 0)
-      (effects (font (size 1.27 1.27)) hide)
-    )
-    (property "Farnell PN" "1972673" (at 151.13 88.9 0)
-      (effects (font (size 1.27 1.27)) hide)
-    )
+    (property "Datasheet" "" (at 151.13 88.9 0)
+      (effects (font (size 1.27 1.27)) (justify left) hide)
+    )
+    (property "LCSC" "C15127" (at 151.13 88.9 0)
+      (effects (font (size 1.27 1.27)) hide)
+    )
+    (property "Farnell PN" "2061518" (at 151.13 88.9 0)
+      (effects (font (size 1.27 1.27)) hide)
+    )
