File: hardware/optiplower.kicad_sch (KiCad schematic)
At the start: 22 parts, among them J1 Conn_01x02, J2 Conn_01x03, U1 LR7533-M, U2 XL4015, U3 DS2502, U4 ATtiny25-10SSU, U5 ATtiny85-20PU, U6 DS2502S+

Commit message: Move PCB into hardware/ folder
Parts:
- U1: now fitted; now in the parts list
Connections:
- net +3V3: now also U1.2 (VO)
- net GND: now also U1.1 (GND)
- net VCC: now also U1.3 (VI)
Other:
- note removed: "Testing shows ATTiny should be run at 2.7v This is a 3v3 part"
Changed lines of the file:
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@@
   (junction (at 182.88 58.42) (diameter 0) (color 0 0 0 0)
+  )
+  (junction (at 227.33 46.99) (diameter 0) (color 0 0 0 0)
   )
   (junction (at 180.34 50.8) (diameter 0) (color 0 0 0 0)
@@
     (stroke (width 0) (type default))
   )
-  (text "Testing shows ATTiny should be run at 2.7v\nThis is a 3v3 part"
-    (at 273.05 29.21 0)
-    (effects (font (size 1.27 1.27)) (justify left bottom))
-  )
   (text "Adjustability from 18.29v - 20.125v" (at 120.65 62.23 0)
     (effects (font (size 1.27 1.27)) (justify left bottom))
@@
     )
   )
-  (symbol (lib_id "Regulator_Linear:AZ1117-3.3") (at 264.16 25.4 0) (unit 1)
-    (in_bom no) (on_board no) (dnp yes) (fields_autoplaced)
-    (property "Reference" "U1" (at 264.16 19.05 0)
-      (effects (font (size 1.27 1.27)))
-    )
-    (property "Value" "LR7533-M" (at 264.16 21.59 0)
-      (effects (font (size 1.27 1.27)))
-    )
-    (property "Footprint" "Package_TO_SOT_SMD:SOT-89-3_Handsoldering" (at 264.16 19.05 0)
+  (symbol (lib_id "Regulator_Linear:AZ1117-3.3") (at 227.33 39.37 0) (unit 1)
+    (in_bom yes) (on_board yes) (dnp no) (fields_autoplaced)
+    (property "Reference" "U1" (at 227.33 33.02 0)
+      (effects (font (size 1.27 1.27)))
+    )
+    (property "Value" "LR7533-M" (at 227.33 35.56 0)
+      (effects (font (size 1.27 1.27)))
+    )
+    (property "Footprint" "Package_TO_SOT_SMD:SOT-89-3_Handsoldering" (at 227.33 33.02 0)
       (effects (font (size 1.27 1.27) italic) hide)
     )
-    (property "Datasheet" "" (at 264.16 25.4 0)
-      (effects (font (size 1.27 1.27)) hide)
-    )
-    (property "LCSC" "C486076" (at 264.16 25.4 0)
-      (effects (font (size 1.27 1.27)) hide)
-    )
-    (property "MPN" "LR7533-M" (at 264.16 25.4 0)
-      (effects (font (size 1.27 1.27)) hide)
-    )
-    (property "Manufacturer" "LR" (at 264.16 25.4 0)
-      (effects (font (size 1.27 1.27)) hide)
-    )
+    (property "Datasheet" "" (at 227.33 39.37 0)
+      (effects (font (size 1.27 1.27)) hide)
+    )
+    (property "LCSC" "C486076" (at 227.33 39.37 0)
+      (effects (font (size 1.27 1.27)) hide)
+    )
+    (property "MPN" "LR7533-M" (at 227.33 39.37 0)
+      (effects (font (size 1.27 1.27)) hide)
+    )
+    (property "Manufacturer" "LR" (at 227.33 39.37 0)
+      (effects (font (size 1.27 1.27)) hide)
+    )
